File: USBU-LDO.kicad_sch (KiCad schematic)
At the start: 7 parts, among them J1 USB_B_Micro, J2 Conn_01x05_Pin, U1 AMS1117-3.3

Commit message: Renamed the board
Other:
- title: USB-LDO-U-0010 -> USBU-LDO-0010
Changed lines of the file:
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@@
   (paper "A4")
   (title_block
-    (title "USB-LDO-U-0010")
-    (date "2024-01-31")
+    (title "USBU-LDO-0010")
+    (date "2024-02-01")
     (rev "1.0")
     (company "(c) Andriy Golovnya")
@@
     (pin "1")
     (instances
-      (project "USB-LDO-U"
+      (project "USBU-LDO"
         (path "/d5c5ffdd-0789-4403-9797-75c531715feb"
           (reference "#PWR06") (unit 1)
@@
     (pin "1")
     (instances
-      (project "USB-LDO-U"
+      (project "USBU-LDO"
         (path "/d5c5ffdd-0789-4403-9797-75c531715feb"
           (reference "#PWR04") (unit 1)
@@
     (pin "1")
     (instances
-      (project "USB-LDO-U"
+      (project "USBU-LDO"
         (path "/d5c5ffdd-0789-4403-9797-75c531715feb"
           (reference "#PWR09") (unit 1)
@@
     (pin "1")
     (instances
-      (project "USB-LDO-U"
+      (project "USBU-LDO"
         (path "/d5c5ffdd-0789-4403-9797-75c531715feb"
           (reference "C2") (unit 1)
@@
     (pin "1")
     (instances
-      (project "USB-LDO-U"
+      (project "USBU-LDO"
         (path "/d5c5ffdd-0789-4403-9797-75c531715feb"
           (reference "#PWR02") (unit 1)
@@
     (pin "1")
     (instances
-      (project "USB-LDO-U"
+      (project "USBU-LDO"
         (path "/d5c5ffdd-0789-4403-9797-75c531715feb"
           (reference "#PWR03") (unit 1)
@@
     (pin "2")
     (instances
-      (project "USB-LDO-U"
+      (project "USBU-LDO"
         (path "/d5c5ffdd-0789-4403-9797-75c531715feb"
           (reference "J1") (unit 1)
@@
     (pin "1")
     (instances
-      (project "USB-LDO-U"
+      (project "USBU-LDO"
         (path "/d5c5ffdd-0789-4403-9797-75c531715feb"
           (reference "#PWR05") (unit 1)
@@
     (pin "2")
     (instances
-      (project "USB-LDO-U"
+      (project "USBU-LDO"
         (path "/d5c5ffdd-0789-4403-9797-75c531715feb"
           (reference "U1") (unit 1)
@@
     (pin "5")
     (instances
-      (project "USB-LDO-U"
+      (project "USBU-LDO"
         (path "/d5c5ffdd-0789-4403-9797-75c531715feb"
           (reference "J2") (unit 1)
@@
     (pin "1")
     (instances
-      (project "USB-LDO-U"
+      (project "USBU-LDO"
         (path "/d5c5ffdd-0789-4403-9797-75c531715feb"
           (reference "D1") (unit 1)
@@
     (pin "1")
     (instances
-      (project "USB-LDO-U"
+      (project "USBU-LDO"
         (path "/d5c5ffdd-0789-4403-9797-75c531715feb"
           (reference "#PWR01") (unit 1)
@@
     (pin "1")
     (instances
-      (project "USB-LDO-U"
+      (project "USBU-LDO"
         (path "/d5c5ffdd-0789-4403-9797-75c531715feb"
           (reference "#PWR011") (unit 1)
@@
     (pin "1")
     (instances
-      (project "USB-LDO-U"
+      (project "USBU-LDO"
         (path "/d5c5ffdd-0789-4403-9797-75c531715feb"
           (reference "C1") (unit 1)
@@
     (pin "1")
     (instances
-      (project "USB-LDO-U"
+      (project "USBU-LDO"
         (path "/d5c5ffdd-0789-4403-9797-75c531715feb"
           (reference "#PWR07") (unit 1)
@@
     (pin "1")
     (instances
-      (project "USB-LDO-U"
+      (project "USBU-LDO"
         (path "/d5c5ffdd-0789-4403-9797-75c531715feb"
           (reference "#PWR08") (unit 1)
@@
     (pin "2")
     (instances
-      (project "USB-LDO-U"
+      (project "USBU-LDO"
         (path "/d5c5ffdd-0789-4403-9797-75c531715feb"
           (reference "R1") (unit 1)
@@
     (pin "1")
     (instances
-      (project "USB-LDO-U"
+      (project "USBU-LDO"
         (path "/d5c5ffdd-0789-4403-9797-75c531715feb"
           (reference "#PWR010") (unit 1)
@@
     (pin "1")
     (instances
-      (project "USB-LDO-U"
+      (project "USBU-LDO"
         (path "/d5c5ffdd-0789-4403-9797-75c531715feb"
           (reference "#PWR012") (unit 1)
